File: pcb/proto1/powersupply.kicad_sch (KiCad schematic)
At the start: 52 parts

Commit message: .
Parts:
- L? (x2): footprint (none) -> Inductor_SMD:L_Taiyo-Yuden_NR-50xx
Changed lines of the file:
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@@
     (property "Reference" "L?" (id 0) (at 186.69 135.89 90))
     (property "Value" "L" (id 1) (at 186.69 138.43 90))
-    (property "Footprint" "" (id 2) (at 186.69 142.24 0)
+    (property "Footprint" "Inductor_SMD:L_Taiyo-Yuden_NR-50xx" (id 2) (at 186.69 142.24 0)
       (effects (font (size 1.27 1.27)) hide)
     )
@@
     (property "Reference" "L?" (id 0) (at 186.69 168.91 90))
     (property "Value" "L" (id 1) (at 186.69 171.45 90))
-    (property "Footprint" "" (id 2) (at 186.69 175.26 0)
-      (effects (font (size 1.27 1.27)) hide)
-    )
+    (property "Footprint" "Inductor_SMD:L_Taiyo-Yuden_NR-50xx" (id 2) (at 186.69 175.26 0)
+      (effects (font (size 1.27 1.27)) hide)
+    )

Commit message: footprints
Parts:
- gave numbers to parts that had none: 52
