File: pcb/proto1/proto1.kicad_pcb (KiCad board)
At the start: 4 copper layers, 182 parts, among them U1 ATSAM4C4, U12 NE5532, U13 NE5532, U15 R1283K, U17 ?, U18 ?, U19 AP7361C-33E, U2 NDS36P, U3 ATSAMD21E17D-A, U4 ATSAMD21E17D-A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

Commit message: .
Parts:
- moved C23 183.9 mm to (110.7, 80.0)
- moved C18 141.2 mm to (93.0, 74.7)
- moved C15 141.2 mm to (97.8, 74.7)
- moved U2 4.49 mm to (172.7, 106.7), turned to 90 degrees
Connections:
- U1 pad 1: unconnected-(U1-Pad1) -> SW_StartPause
- U1 pad 19: /RAS -> unconnected-(U1-Pad19)
- U1 pad 2: unconnected-(U1-Pad2) -> SW_Stop
- U1 pad 20: /CAS -> unconnected-(U1-Pad20)
- U1 pad 21: /WE -> unconnected-(U1-Pad21)
- U1 pad 24: /CLK -> unconnected-(U1-Pad24)
- U1 pad 29: SW_Restart -> unconnected-(U1-Pad29)
- U1 pad 3: unconnected-(U1-Pad3) -> SW_Restart
- U1 pad 31: SW_Stop -> unconnected-(U1-Pad31)
- U1 pad 32: SW_LoopInc -> unconnected-(U1-Pad32)
- U1 pad 43: SW_LoopIn -> /CS
- U1 pad 45: SW_LoopOut -> /RAS
- U1 pad 46: SW_LoopDec -> /CAS
- U1 pad 47: SW_StartPause -> /WE
- U1 pad 5: unconnected-(U1-Pad5) -> SW_Reverse
- U1 pad 52: (no net) -> GND
- U1 pad 54: SW_Reverse -> unconnected-(U1-Pad54)
- U1 pad 59: /CS -> unconnected-(U1-Pad59)
- U1 pad 6: unconnected-(U1-Pad6) -> SW_LoopDec
- U1 pad 60: /DQ7 -> /DQ0
- U1 pad 61: /DQ6 -> /DQ1
- U1 pad 64: /DQ5 -> /DQ2
- U1 pad 65: /DQ4 -> /DQ3
- U1 pad 66: /DQ3 -> /DQ4
- U1 pad 67: /DQ2 -> /DQ5
- U1 pad 68: /DQ1 -> /DQ6
- U1 pad 69: /DQ0 -> /DQ7
- U1 pad 7: unconnected-(U1-Pad7) -> SW_LoopOut
- U1 pad 70: /DQ15 -> /DQ8
- U1 pad 71: /DQ14 -> /DQ9
- U1 pad 72: /DQ13 -> /DQ10
- U1 pad 73: /DQ12 -> /DQ11
- U1 pad 74: /DQ11 -> /DQ12
- U1 pad 75: /DQ10 -> /DQ13
- U1 pad 79: /DQ9 -> /DQ15
- U1 pad 8: unconnected-(U1-Pad8) -> SW_LoopIn
- U1 pad 80: /DQ8 -> /DQ14
- U1 pad 81: unconnected-(U1-Pad81) -> /CLK
- U1 pad 83: unconnected-(U1-Pad83) -> /CKE
- U1 pad 84: /CKE -> /A12
- U1 pad 87: unconnected-(U1-Pad87) -> /A11
- U1 pad 88: unconnected-(U1-Pad88) -> /A9
- U1 pad 9: unconnected-(U1-Pad9) -> SW_LoopInc
- U1 pad 90: unconnected-(U1-Pad90) -> /A8
- U1 pad 91: unconnected-(U1-Pad91) -> /A7
- U1 pad 93: unconnected-(U1-Pad93) -> /A6
- U1 pad 94: unconnected-(U1-Pad94) -> /A5
- U1 pad 95: unconnected-(U1-Pad95) -> /A4
Routing:
- net /A4: track 0.00 -> 46.9 mm
- net /A5: track 0.00 -> 44.9 mm
- net /A6: track 0.00 -> 43.2 mm
- net /A7: track 0.00 -> 41.1 mm
- net /A8: track 0.00 -> 39.3 mm
- net /A9: track 0.00 -> 37.3 mm
- net /A11: track 0.00 -> 35.5 mm
- net /A12: track 0.00 -> 33.1 mm
- net /CS: track 0.00 -> 31.4 mm
- net /CKE: track 0.00 -> 31.3 mm
- net /RAS: track 0.00 -> 29.3 mm
- net /CLK: track 0.00 -> 29.3 mm
- net /CAS: track 0.00 -> 27.4 mm
- net /WE: track 0.00 -> 25.6 mm
- net /DQ7: track 0.00 -> 23.0 mm
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Other:
- board outline added: 191.8 x 114.3 mm

Commit message: ..
Parts:
- moved U2 1.27 mm to (172.7, 105.4)
- turned U1 to 180 degrees
Connections:
- U1 pad 1: SW_StartPause -> /DQ2
- U1 pad 10: unconnected-(U1-Pad10) -> /A5
- U1 pad 12: unconnected-(U1-Pad12) -> /A6
- U1 pad 13: unconnected-(U1-Pad13) -> /A8
- U1 pad 14: unconnected-(U1-Pad14) -> /A9
- U1 pad 15: unconnected-(U1-Pad15) -> /A11
- U1 pad 16: unconnected-(U1-Pad16) -> /A12
- U1 pad 17: unconnected-(U1-Pad17) -> /DQ8
- U1 pad 18: unconnected-(U1-Pad18) -> /DQ9
- U1 pad 19: unconnected-(U1-Pad19) -> /DQ10
- U1 pad 2: SW_Stop -> /DQ1
- U1 pad 20: unconnected-(U1-Pad20) -> /DQ11
- U1 pad 21: unconnected-(U1-Pad21) -> /DQ12
- U1 pad 22: /LDQM -> /DQ13
- U1 pad 23: /UDQM -> /DQ14
- U1 pad 24: unconnected-(U1-Pad24) -> /DQ15
- U1 pad 29: unconnected-(U1-Pad29) -> /CLK
- U1 pad 3: SW_Restart -> /DQ0
- U1 pad 43: /CS -> unconnected-(U1-Pad43)
- U1 pad 45: /RAS -> unconnected-(U1-Pad45)
- U1 pad 46: /CAS -> unconnected-(U1-Pad46)
- U1 pad 47: /WE -> unconnected-(U1-Pad47)
- U1 pad 5: SW_Reverse -> /A0
- U1 pad 6: SW_LoopDec -> /A1
- U1 pad 60: /DQ0 -> unconnected-(U1-Pad60)
- U1 pad 61: /DQ1 -> unconnected-(U1-Pad61)
- U1 pad 64: /DQ2 -> unconnected-(U1-Pad64)
- U1 pad 65: /DQ3 -> unconnected-(U1-Pad65)
- U1 pad 66: /DQ4 -> unconnected-(U1-Pad66)
- U1 pad 67: /DQ5 -> unconnected-(U1-Pad67)
- U1 pad 68: /DQ6 -> unconnected-(U1-Pad68)
- U1 pad 69: /DQ7 -> unconnected-(U1-Pad69)
- U1 pad 7: SW_LoopOut -> /A2
- U1 pad 70: /DQ8 -> unconnected-(U1-Pad70)
- U1 pad 71: /DQ9 -> unconnected-(U1-Pad71)
- U1 pad 72: /DQ10 -> unconnected-(U1-Pad72)
- U1 pad 73: /DQ11 -> unconnected-(U1-Pad73)
- U1 pad 74: /DQ12 -> unconnected-(U1-Pad74)
- U1 pad 75: /DQ13 -> unconnected-(U1-Pad75)
- U1 pad 79: /DQ15 -> unconnected-(U1-Pad79)
- U1 pad 8: SW_LoopIn -> /A3
- U1 pad 80: /DQ14 -> unconnected-(U1-Pad80)
- U1 pad 81: /CLK -> unconnected-(U1-Pad81)
- U1 pad 83: /CKE -> unconnected-(U1-Pad83)
- U1 pad 84: /A12 -> unconnected-(U1-Pad84)
- U1 pad 87: /A11 -> unconnected-(U1-Pad87)
- U1 pad 88: /A9 -> unconnected-(U1-Pad88)
- U1 pad 9: SW_LoopInc -> /A4
- U1 pad 90: /A8 -> unconnected-(U1-Pad90)
- U1 pad 91: /A7 -> unconnected-(U1-Pad91)
- U1 pad 93: /A6 -> unconnected-(U1-Pad93)
- U1 pad 94: /A5 -> unconnected-(U1-Pad94)
- U1 pad 95: /A4 -> unconnected-(U1-Pad95)
Routing:
- net /A7: track 41.1 -> 0.00 mm
- net /CS: track 31.4 -> 0.00 mm
- net /CKE: track 31.3 -> 0.00 mm
- net /RAS: track 29.3 -> 0.00 mm
- net /A3: track 0.00 -> 29.3 mm
- net /A2: track 0.00 -> 28.4 mm
- net /CAS: track 27.4 -> 0.00 mm
- net /A1: track 0.00 -> 27.4 mm
- net /A0: track 0.00 -> 26.4 mm
- net /WE: track 25.6 -> 0.00 mm
- net /DQ7: track 23.0 -> 0.00 mm
- net /DQ6: track 21.8 -> 0.00 mm
- net /DQ5: track 20.8 -> 0.00 mm
- net /DQ4: track 17.9 -> 0.00 mm
- net /DQ3: track 17.0 -> 0.00 mm
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
Commit message: Update
Connections:
- U1 pad 10: /A5 -> /A6
- U1 pad 100: unconnected-(U1-Pad100) -> /DQ3
- U1 pad 12: /A6 -> /A7
- U1 pad 5: /A0 -> /A1
- U1 pad 6: /A1 -> /A2
- U1 pad 7: /A2 -> /A3
- U1 pad 8: /A3 -> /A4
- U1 pad 81: unconnected-(U1-Pad81) -> /A0
- U1 pad 83: unconnected-(U1-Pad83) -> /A10
- U1 pad 84: unconnected-(U1-Pad84) -> /BA1
- U1 pad 87: unconnected-(U1-Pad87) -> /BA0
- U1 pad 88: unconnected-(U1-Pad88) -> /CS
- U1 pad 9: /A4 -> /A5
- U1 pad 90: unconnected-(U1-Pad90) -> /RAS
- U1 pad 91: unconnected-(U1-Pad91) -> /CAS
- U1 pad 93: unconnected-(U1-Pad93) -> /WE
- U1 pad 94: unconnected-(U1-Pad94) -> /DQ7
- U1 pad 95: unconnected-(U1-Pad95) -> /DQ6
- U1 pad 96: unconnected-(U1-Pad96) -> /DQ5
- U1 pad 97: unconnected-(U1-Pad97) -> /DQ4
Routing:
- net /A10: track 0.00 -> 42.2 mm
- net /BA1: track 0.00 -> 40.4 mm
- net /BA0: track 0.00 -> 38.2 mm
- net /CS: track 0.00 -> 36.5 mm
- net /RAS: track 0.00 -> 34.6 mm
- net /CAS: track 0.00 -> 32.8 mm
- net /WE: track 0.00 -> 30.3 mm
- net /A7: track 0.00 -> 28.7 mm
- net /DQ7: track 0.00 -> 27.0 mm
- net /DQ6: track 0.00 -> 24.4 mm
- net /DQ5: track 0.00 -> 22.6 mm
- net /DQ4: track 0.00 -> 20.1 mm
- net /A0: track 26.4 -> 45.9 mm
- net /DQ3: track 0.00 -> 15.9 mm
