File: pcb/proto1/proto1.kicad_sch (KiCad schematic)
At the start: 166 parts

Commit message: footprints
Parts:
- U1: renamed from U?; footprint (none) -> Package_QFP:LQFP-100_14x14mm_P0.5mm
- U12, U13, U5, U7, U9: renamed from U?; footprint (none) -> Package_SO:SOIC-8_3.9x4.9mm_P1.27mm
- U2: renamed from U?; footprint (none) -> Package_SO:TSOP-II-54_22.2x10.16mm_P0.8mm
- gave numbers to parts that had none: 151
Connections:
- net A0: no longer U1.64 (PA3)
- net A1: no longer U1.83 (PA4/AD1)
- net A10: no longer U1.65 (PA21)
- net A11: no longer U1.66 (PA22)
- net A12: no longer U1.67 (PA23)
- net A2: no longer U1.68 (PA9)
- net A3: no longer U1.69 (PA10)
- net A4: no longer U1.70 (PA11)
- net A5: no longer U1.71 (PA13)
- net A6: no longer U1.72 (PA14)
- net A7: no longer U1.73 (PA15)
- net A8: no longer U1.74 (PA16)
- net A9: no longer U1.75 (PA17)
- net BA0: no longer U1.61 (PA27)
- net BA1: no longer U1.60 (PA28)
- net DQ0: now also U1.69 (PA10); no longer U1.1 (PB6)
- net DQ1: now also U1.68 (PA9); no longer U1.2 (PB7)
- net DQ10: now also U1.75 (PA17); no longer U1.5 (PB19)
- net DQ11: now also U1.74 (PA16); no longer U1.7 (PB22)
- net DQ12: now also U1.73 (PA15); no longer U1.10 (PB24)
- net DQ13: now also U1.72 (PA14); no longer U1.9 (PB25)
- net DQ14: now also U1.71 (PA13); no longer U1.12 (PB29)
- net DQ15: now also U1.70 (PA11); no longer U1.8 (PB30)
- net DQ2: now also U1.67 (PA23); no longer U1.6 (PB8)
- net DQ3: now also U1.66 (PA22); no longer U1.13 (PB9)
- net DQ4: now also U1.65 (PA21); no longer U1.14 (PB10)
- net DQ5: now also U1.64 (PA3); no longer U1.15 (PB11)
- net DQ6: now also U1.61 (PA27); no longer U1.16 (PB12)
- net DQ7: now also U1.60 (PA28); no longer U1.17 (PB14)
- net DQ8: now also U1.80 (PB23/AD4); no longer U1.18 (PB15)
- net DQ9: now also U1.79 (PB31/AD5); no longer U1.3 (PB18)
- no-connect marks 49 -> 47

Commit message: .
Connections:
- net A11: now also U1.87 (PB21)
- net A12: now also U1.84 (PA12/AD0)
- net A4: now also U1.95 (PB16)
- net A5: now also U1.94 (PB28)
- net A6: now also U1.93 (PB26)
- net A7: now also U1.91 (PB27)
- net A8: now also U1.90 (PA0)
- net A9: now also U1.88 (PB20)
- net CAS: now also U1.46 (PC7); no longer U1.20 (PA25)
- net CKE: now also U1.83 (PA4/AD1); no longer U1.84 (PA12/AD0)
- net CLK: now also U1.81 (PB13/AD3); no longer U1.24 (PA18)
- net CS: now also U1.43 (PB4); no longer U1.59 (PA29)
- net DQ0: now also U1.60 (PA28); no longer U1.69 (PA10)
- net DQ1: now also U1.61 (PA27); no longer U1.68 (PA9)
- net DQ10: now also U1.72 (PA14); no longer U1.75 (PA17)
- net DQ11: now also U1.73 (PA15); no longer U1.74 (PA16)
- net DQ12: now also U1.74 (PA16); no longer U1.73 (PA15)
- net DQ13: now also U1.75 (PA17); no longer U1.72 (PA14)
- net DQ14: now also U1.80 (PB23/AD4); no longer U1.71 (PA13)
- net DQ15: now also U1.79 (PB31/AD5); no longer U1.70 (PA11)
- net DQ2: now also U1.64 (PA3); no longer U1.67 (PA23)
- net DQ3: now also U1.65 (PA21); no longer U1.66 (PA22)
- net DQ4: now also U1.66 (PA22); no longer U1.65 (PA21)
- net DQ5: now also U1.67 (PA23); no longer U1.64 (PA3)
- net DQ6: now also U1.68 (PA9); no longer U1.61 (PA27)
- net DQ7: now also U1.69 (PA10); no longer U1.60 (PA28)
- net DQ8: now also U1.70 (PA11); no longer U1.80 (PB23/AD4)
- net DQ9: now also U1.71 (PA13); no longer U1.79 (PB31/AD5)
- net GND: now also U1.52 (GND)
- net RAS: now also U1.45 (PB5); no longer U1.19 (PA26)
- net SW_LoopDec: now also U1.6 (PB8); no longer U1.46 (PC7)
- net SW_LoopIn: now also U1.8 (PB30); no longer U1.43 (PB4)
- net SW_LoopInc: now also U1.9 (PB25); no longer U1.32 (PC6)
- net SW_LoopOut: now also U1.7 (PB22); no longer U1.45 (PB5)
- net SW_Restart: now also U1.3 (PB18); no longer U1.29 (PC9)
- net SW_Reverse: now also U1.5 (PB19); no longer U1.54 (PC8)
- net SW_StartPause: now also U1.1 (PB6); no longer U1.47 (PC0)
- net SW_Stop: now also U1.2 (PB7); no longer U1.31 (PC1)
- net WE: now also U1.47 (PC0); no longer U1.21 (PA24)
- no-connect marks 47 -> 36

Commit message: ..
Connections:
- net A0: now also U1.5 (PB19)
- net A1: now also U1.6 (PB8)
- net A11: now also U1.15 (PB11); no longer U1.87 (PB21)
- net A12: now also U1.16 (PB12); no longer U1.84 (PA12/AD0)
- net A2: now also U1.7 (PB22)
- net A3: now also U1.8 (PB30)
- net A4: now also U1.9 (PB25); no longer U1.95 (PB16)
- net A5: now also U1.10 (PB24); no longer U1.94 (PB28)
- net A6: now also U1.12 (PB29); no longer U1.93 (PB26)
- net A7: no longer U1.91 (PB27)
- net A8: now also U1.13 (PB9); no longer U1.90 (PA0)
- net A9: now also U1.14 (PB10); no longer U1.88 (PB20)
- net CAS: no longer U1.46 (PC7)
- net CKE: no longer U1.83 (PA4/AD1)
- net CLK: now also U1.29 (PC9); no longer U1.81 (PB13/AD3)
- net CS: no longer U1.43 (PB4)
- net DQ0: now also U1.3 (PB18); no longer U1.60 (PA28)
- net DQ1: now also U1.2 (PB7); no longer U1.61 (PA27)
- net DQ10: now also U1.19 (PA26); no longer U1.72 (PA14)
- net DQ11: now also U1.20 (PA25); no longer U1.73 (PA15)
- net DQ12: now also U1.21 (PA24); no longer U1.74 (PA16)
- net DQ13: now also U1.22 (PA20); no longer U1.75 (PA17)
- net DQ14: now also U1.23 (PA19); no longer U1.80 (PB23/AD4)
- net DQ15: now also U1.24 (PA18); no longer U1.79 (PB31/AD5)
- net DQ2: now also U1.1 (PB6); no longer U1.64 (PA3)
- net DQ3: no longer U1.65 (PA21)
- net DQ4: no longer U1.66 (PA22)
- net DQ5: no longer U1.67 (PA23)
- net DQ6: no longer U1.68 (PA9)
- net DQ7: no longer U1.69 (PA10)
- net DQ8: now also U1.17 (PB14); no longer U1.70 (PA11)
- net DQ9: now also U1.18 (PB15); no longer U1.71 (PA13)
- net LDQM: no longer U1.22 (PA20)
- net RAS: no longer U1.45 (PB5)
- net SW_LoopDec: no longer U1.6 (PB8)
- net SW_LoopIn: no longer U1.8 (PB30)
- net SW_LoopInc: no longer U1.9 (PB25)
- net SW_LoopOut: no longer U1.7 (PB22)
- net SW_Restart: no longer U1.3 (PB18)
- net SW_Reverse: no longer U1.5 (PB19)
- net SW_StartPause: no longer U1.1 (PB6)
- net SW_Stop: no longer U1.2 (PB7)
- net UDQM: no longer U1.23 (PA19)
- net WE: no longer U1.47 (PC0)

Commit message: Update
Connections:
- net A0: now also U1.81 (PB13/AD3); no longer U1.5 (PB19)
- net A1: now also U1.5 (PB19); no longer U1.6 (PB8)
- net A10: now also U1.83 (PA4/AD1)
- net A2: now also U1.6 (PB8); no longer U1.7 (PB22)
- net A3: now also U1.7 (PB22); no longer U1.8 (PB30)
- net A4: now also U1.8 (PB30); no longer U1.9 (PB25)
- net A5: now also U1.9 (PB25); no longer U1.10 (PB24)
- net A6: now also U1.10 (PB24); no longer U1.12 (PB29)
- net A7: now also U1.12 (PB29)
- net BA0: now also U1.87 (PB21)
- net BA1: now also U1.84 (PA12/AD0)
- net CAS: now also U1.91 (PB27)
- net CS: now also U1.88 (PB20)
- net DQ3: now also U1.100 (PA2)
- net DQ4: now also U1.97 (PB17)
- net DQ5: now also U1.96 (PA1)
- net DQ6: now also U1.95 (PB16)
- net DQ7: now also U1.94 (PB28)
- net RAS: now also U1.90 (PA0)
- net WE: now also U1.93 (PB26)
Changed lines of the file:
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@@
     (effects (font (size 1.27 1.27)) (justify left bottom))
+  )
+  (label "BA1" (at 76.2 542.29 180)
+    (effects (font (size 1.27 1.27)) (justify right bottom))
   )
   (label "A3" (at 86.36 673.1 180)
@@
     (effects (font (size 1.27 1.27)) (justify right bottom))
   )
-  (label "DQ7" (at 134.62 543.56 0)
+  (label "DQ7" (at 119.38 582.93 0)
     (effects (font (size 1.27 1.27)) (justify left bottom))
   )
@@
     (effects (font (size 1.27 1.27)) (justify left bottom))
   )
-  (label "DQ4" (at 134.62 530.86 0)
-    (effects (font (size 1.27 1.27)) (justify left bottom))
-  )
-  (label "DQ0" (at 135.89 588.01 0)
+  (label "DQ4" (at 119.38 554.99 0)
     (effects (font (size 1.27 1.27)) (justify left bottom))
   )
@@
     (effects (font (size 1.27 1.27)) (justify left bottom))
   )
-  (label "A1" (at 119.38 532.13 0)
+  (label "A2" (at 119.38 532.13 0)
     (effects (font (size 1.27 1.27)) (justify left bottom))
   )
@@
     (effects (font (size 1.27 1.27)) (justify left bottom))
   )
+  (label "RAS" (at 76.2 511.81 180)
+    (effects (font (size 1.27 1.27)) (justify right bottom))
+  )
   (label "DQ0" (at 119.38 557.53 0)
     (effects (font (size 1.27 1.27)) (justify left bottom))
@@
     (effects (font (size 1.27 1.27)) (justify left bottom))
   )
-  (label "A5" (at 119.38 572.77 0)
+  (label "A6" (at 119.38 572.77 0)
     (effects (font (size 1.27 1.27)) (justify left bottom))
   )
@@
     (effects (font (size 1.27 1.27)) (justify right bottom))
   )
-  (label "A4" (at 119.38 575.31 0)
+  (label "A5" (at 119.38 575.31 0)
     (effects (font (size 1.27 1.27)) (justify left bottom))
   )
@@
     (effects (font (size 1.27 1.27)) (justify right bottom))
   )
-  (label "A0" (at 119.38 560.07 0)
+  (label "CAS" (at 119.38 580.39 0)
+    (effects (font (size 1.27 1.27)) (justify left bottom))
+  )
+  (label "A1" (at 119.38 560.07 0)
     (effects (font (size 1.27 1.27)) (justify left bottom))
   )
@@
     (effects (font (size 1.27 1.27)) (justify left bottom))
   )
+  (label "BA0" (at 119.38 565.15 0)
+    (effects (font (size 1.27 1.27)) (justify left bottom))
+  )
   (label "DQ13" (at 116.84 698.5 0)
     (effects (font (size 1.27 1.27)) (justify left bottom))
   )
+  (label "A10" (at 76.2 521.97 180)
+    (effects (font (size 1.27 1.27)) (justify right bottom))
+  )
   (label "LDQM" (at 86.36 712.47 180)
     (effects (font (size 1.27 1.27)) (justify right bottom))
   )
-  (label "A6" (at 119.38 585.47 0)
+  (label "A7" (at 119.38 585.47 0)
     (effects (font (size 1.27 1.27)) (justify left bottom))
   )
@@
     (effects (font (size 1.27 1.27)) (justify right bottom))
   )
+  (label "CS" (at 119.38 562.61 0)
+    (effects (font (size 1.27 1.27)) (justify left bottom))
+  )
   (label "A12" (at 119.38 542.29 0)
     (effects (font (size 1.27 1.27)) (justify left bottom))
   )
-  (label "DQ1" (at 133.35 579.12 0)
-    (effects (font (size 1.27 1.27)) (justify left bottom))
-  )
-  (label "A2" (at 119.38 567.69 0)
+  (label "A0" (at 119.38 544.83 0)
+    (effects (font (size 1.27 1.27)) (justify left bottom))
+  )
+  (label "A3" (at 119.38 567.69 0)
     (effects (font (size 1.27 1.27)) (justify left bottom))
   )
@@
     (effects (font (size 1.27 1.27)) (justify left bottom))
   )
+  (label "WE" (at 119.38 577.85 0)
+    (effects (font (size 1.27 1.27)) (justify left bottom))
+  )
   (label "A10" (at 86.36 690.88 180)
     (effects (font (size 1.27 1.27)) (justify right bottom))
@@
     (effects (font (size 1.27 1.27)) (justify left bottom))
   )
-  (label "DQ6" (at 135.89 538.48 0)
+  (label "DQ6" (at 119.38 552.45 0)
     (effects (font (size 1.27 1.27)) (justify left bottom))
   )
@@
     (effects (font (size 1.27 1.27)) (justify right bottom))
   )
-  (label "A3" (at 119.38 588.01 0)
+  (label "A4" (at 119.38 588.01 0)
     (effects (font (size 1.27 1.27)) (justify left bottom))
   )
@@
     (effects (font (size 1.27 1.27)) (justify right bottom))
   )
-  (label "DQ2" (at 133.35 568.96 0)
-    (effects (font (size 1.27 1.27)) (justify left bottom))
-  )
   (label "DQ1" (at 119.38 529.59 0)
     (effects (font (size 1.27 1.27)) (justify left bottom))
@@
     (effects (font (size 1.27 1.27)) (justify right bottom))
   )
-  (label "DQ3" (at 135.89 575.31 0)
-    (effects (font (size 1.27 1.27)) (justify left bottom))
-  )
-  (label "DQ5" (at 134.62 534.67 0)
-    (effects (font (size 1.27 1.27)) (justify left bottom))
+  (label "DQ3" (at 76.2 516.89 180)
+    (effects (font (size 1.27 1.27)) (justify right bottom))
+  )
+  (label "DQ5" (at 76.2 514.35 180)
+    (effects (font (size 1.27 1.27)) (justify right bottom))
   )
   (label "DQ15" (at 116.84 703.58 0)
